File: kicad/devboardrp2040.kicad_pcb (KiCad board)
At the start: 4 copper layers, 38.5 x 38.5 mm, 43 parts, among them SW1 SW_Push, SW2 SW_Push, U1 AP63203WU-7, U2 GT-USB-7010ASV, U3 RP2350A_C42411118, U4 W25Q64JVSSIQ_C179171, U5 ABM8-272-T3_C20625731

Commit message: hiii
Parts:
- removed U3: RP2350A_C42411118, easyeda2kicad:QFN-60_L7.0-W7.0-P0.40-TL-EP3.4
- added J1: Conn_01x12_Pin, Connector_PinHeader_2.54mm:PinHeader_1x12_P2.54mm_Vertical, F.Cu at (51.1, 59.7)
- added U6: RP2350A-QFN60, Package_DFN_QFN:QFN-60-1EP_7x7mm_P0.4mm_EP3.4x3.4mm, F.Cu at (78.2, 22.2)
- moved C13 41.5 mm to (53.5, 34.2)
- moved C11 30.2 mm to (70.6, 18.9)
- moved C1 29.6 mm to (62.9, 29.1)
- moved C22 29.2 mm to (59.2, 28.3)
- moved C23 29.2 mm to (59.2, 30.2)
- moved C14 29.2 mm to (56.3, 24.3)
- moved C16 29.2 mm to (56.3, 28.3)
- moved C17 29.2 mm to (56.3, 30.2)
- moved C18 29.2 mm to (56.3, 32.2)
- moved C19 29.2 mm to (56.3, 34.2)
- moved C20 29.2 mm to (59.2, 24.3)
- moved C21 29.2 mm to (59.2, 26.3)
- moved C24 29.2 mm to (59.2, 32.2)
- moved C15 29.2 mm to (56.3, 26.3)
- moved C10 29.2 mm to (53.5, 28.3)
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Connections:
- net VREG_AVDD renamed Net-(U6-VREG_AVDD)
- net VREG_PGND renamed GND
- U4 pad 5: Net-(U3-QSPI_SD0) -> IO0
- U4 pad 7: Net-(U3-QSPI_SD3) -> IO3
Routing:
- added copper zone on In1.Cu, net (none)
- added copper zone on In2.Cu, net +3V3
Other:
- board outline removed
