File: kicad/devboardrp2040.kicad_sch (KiCad schematic)
At the start: 41 parts, among them SW1 SW_Push, SW2 SW_Push, U1 AP63203WU-7, U2 GT-USB-7010ASV, U3 RP2350A_C42411118, U4 W25Q64JVSSIQ_C179171, U5 ABM8-272-T3_C20625731

Commit message: updated the kicad files
Parts:
- added D1: LED, LED_SMD:LED_0402_1005Metric, symbol Device:LED
- added R9: 33, Resistor_SMD:R_0402_1005Metric, symbol Device:R
- C1: footprint (none) -> Capacitor_SMD:C_0805_2012Metric
- C10, C11, C12, C13, C14, C15, C16, C17, C18, C19, C2, C20, C21, C22, C23, C24, C8: footprint (none) -> Capacitor_SMD:C_0402_1005Metric
- C3, C4, C5, C6, C7, C9: footprint (none) -> Capacitor_SMD:C_0603_1608Metric
- L1: value L -> 47uh; footprint (none) -> Inductor_SMD:L_1210_3225Metric
- L2: footprint (none) -> Inductor_SMD:L_0805_2012Metric
- R1, R2, R3, R4, R5, R6, R7, R8: footprint (none) -> Resistor_SMD:R_0402_1005Metric
- SW1, SW2: footprint (none) -> Button_Switch_Keyboard:SW_Cherry_MX_1.00u_PCB
Connections:
- net GND: now also U3.61 (GND), D1.1 (K)
- net at U3.37 (GPIO25): now also R9.1
- new net: D1.2 (A), R9.2
Other:
- moved on the sheet: R8, SW2

Commit message: hiii
Parts:
- removed U3: RP2350A_C42411118, easyeda2kicad:QFN-60_L7.0-W7.0-P0.40-TL-EP3.4, symbol EasyEda:RP2350A_C42411118
- added J1, J2: Conn_01x12_Pin, Connector_PinHeader_2.54mm:PinHeader_1x12_P2.54mm_Vertical, symbol Connector:Conn_01x12_Pin
- added U6: RP2350A-QFN60, Package_DFN_QFN:QFN-60-1EP_7x7mm_P0.4mm_EP3.4x3.4mm, symbol RPI:RP2350A-QFN60
Connections:
- net +1V1: now also U6.23 (DVDD), U6.39 (DVDD), U6.50 (VREG_FB), U6.6 (DVDD)
- net +3V3: now also J2.11 (Pin_11), U6.1 (IOVDD), U6.11 (IOVDD), U6.20 (IOVDD), U6.30 (IOVDD), U6.38 (IOVDD), U6.44 (ADC_AVDD), U6.45 (IOVDD), U6.49 (VREG_VIN), U6.53 (USB_OTP_VDD), U6.54 (QSPI_IOVDD)
- net GND: now also J1.1 (Pin_1), J1.12 (Pin_12), J2.1 (Pin_1), J2.12 (Pin_12), U6.47 (VREG_PGND), U6.61 (GND)
- net IO1: now also U6.59 (QSPI_SD1)
- net IO2: now also U6.58 (QSPI_SD2)
- net RUN: now also U6.26 (RUN)
- net USB_VBUS: now also J2.10 (Pin_10)
- net XIN: now also U6.21 (XIN)
- net XOUT: now also U6.22 (XOUT)
- net at R7.1: now also U6.52 (USB_DP)
- net at L2.2: now also U6.48 (VREG_LX)
- net at R9.1: now also U6.37 (GPIO25)
- net at R6.2: now also U6.51 (USB_DM)
- net IO3: now reaches U4.7 (HOLD#orRESET#(IO3))
- net IO3: now also U6.55 (QSPI_SD3)
- net at U4.6 (CLK): now also U6.56 (QSPI_SCLK)
- net IO0: now reaches U4.5 (DI(IO0))
- net IO0: now also U6.57 (QSPI_SD0)
- net VREG_AVDD: no longer names the net of C7.2, R2.2
- net VREG_AVDD: now also U6.46 (VREG_AVDD)
- new net: J1.10 (Pin_10), U6.3 (GPIO1)
- new net: J1.11 (Pin_11), U6.2 (GPIO0)
- new net: J1.2 (Pin_2), U6.13 (GPIO9)
- new net: J1.3 (Pin_3), U6.12 (GPIO8)
- new net: J1.4 (Pin_4), U6.10 (GPIO7)
- new net: J1.5 (Pin_5), U6.9 (GPIO6)
- new net: J1.6 (Pin_6), U6.8 (GPIO5)
- new net: J1.7 (Pin_7), U6.7 (GPIO4)
- new net: J1.8 (Pin_8), U6.5 (GPIO3)
- new net: J1.9 (Pin_9), U6.4 (GPIO2)
- new net: J2.2 (Pin_2), U6.43 (GPIO29_ADC3)
- new net: J2.3 (Pin_3), U6.42 (GPIO28_ADC2)
- new net: J2.4 (Pin_4), U6.41 (GPIO27_ADC1)
- new net: J2.5 (Pin_5), U6.40 (GPIO26_ADC0)
- new net GPIO11: J2.9 (Pin_9), U6.15 (GPIO11)
- new net GPIO12: J2.8 (Pin_8), U6.16 (GPIO12)
- new net GPIO13: J2.7 (Pin_7), U6.17 (GPIO13)
- new net GPIO14: J2.6 (Pin_6), U6.18 (GPIO14)
Other:
- moved on the sheet: C10, C11, C12, C13, C14, C15, C16, C17, C18, C19, C20, C21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
