File: kicad/devboardrp2040.kicad_sch (KiCad schematic)
At the start: 41 parts, among them J1 Conn_01x12_Pin, J2 Conn_01x12_Pin, SW1 SW_Push, SW2 SW_Push, U1 AP63203WU-7, U2 GT-USB-7010ASV, U4 W25Q64JVSSIQ_C179171, U5 ABM8-272-T3_C20625731, U6 RP2350A-QFN60

Commit message: hiii
Parts:
- removed J1, J2: Conn_01x12_Pin, Connector_PinHeader_2.54mm:PinHeader_1x12_P2.54mm_Vertical, symbol Connector:Conn_01x12_Pin
- removed R8: 1k, Resistor_SMD:R_0402_1005Metric, symbol Device:R
- removed SW2: SW_Push, easyeda2kicad:SW-SMD_L3.9-W3.0-P4.45, symbol Switch:SW_Push
- added D1: LED, LED_SMD:LED_0402_1005Metric, symbol Device:LED
- added J1, J2: Conn_01x23_Pin, Connector_PinHeader_2.54mm:PinHeader_1x23_P2.54mm_Vertical, symbol Connector:Conn_01x23_Pin
- added R9: 33, Resistor_SMD:R_0402_1005Metric, symbol Device:R
- added SW3, SW4: SW_Push, Button_Switch_Keyboard:SW_Cherry_MX_1.00u_Plate, symbol Switch:SW_Push
- SW1: footprint easyeda2kicad:SW-SMD_L3.9-W3.0-P4.45 -> Button_Switch_Keyboard:SW_Cherry_MX_1.00u_Plate
Connections:
- net GND: now also D1.1 (K), J1.1 (Pin_1), J1.11 (Pin_11), J1.16 (Pin_16), J1.21 (Pin_21), J1.6 (Pin_6), J2.1 (Pin_1), J2.11 (Pin_11), J2.16 (Pin_16), J2.21 (Pin_21), J2.6 (Pin_6), SW3.2, SW4.1
- net GPIO11: now also R4.2, SW1.2
- net at R3.1, R4.1, U4.1 (~{CS}): now also U6.60 (QSPI_SS)
- net at U6.28 (GPIO17): now also SW3.1
- net at U6.29 (GPIO18): now also SW4.2
- net at U6.37 (GPIO25): now also R9.1
- new net: D1.2 (A), R9.2

Commit message: FINISHED KAUHdiodu
Parts:
- L1: value 47uh -> 3.9uh
Connections:
- net +1V1: now also J1.2 (Pin_2)
- net +3V3: now also J1.23 (Pin_23), J2.23 (Pin_23)
- net GND: now also J1.3 (Pin_3), J2.4 (Pin_4)
- net GPIO11: now also J1.18 (Pin_18)
- net GPIO12: now also J1.19 (Pin_19)
- net GPIO20: now also J2.13 (Pin_13)
- net GPIO24: now also J2.7 (Pin_7)
- net RUN: now also J1.20 (Pin_20)
- net USB_VBUS: now also J1.22 (Pin_22), J2.22 (Pin_22)
- net GPIO21: now reaches J2.10 (Pin_10)
- net GPIO21: now also U6.33 (GPIO21)
- net GPIO19: now reaches J2.12 (Pin_12)
- net GPIO19: now also U6.31 (GPIO19)
- net GPIO16: now reaches J2.14 (Pin_14)
- net GPIO16: now also U6.27 (GPIO16)
- net SWDIO: now reaches J2.15 (Pin_15)
- net SWDIO: now also U6.25 (SWDIO)
- net SWCLK: now reaches J2.17 (Pin_17)
- net SWCLK: now also U6.24 (SWCLK)
- net GPIO15: now reaches J2.18 (Pin_18)
- net GPIO15: now also U6.19 (GPIO15)
- net GPIO14: now reaches J2.19 (Pin_19)
- net GPIO14: now also U6.18 (GPIO14)
- net GPIO29: now reaches J2.2 (Pin_2)
- net GPIO29: now also U6.43 (GPIO29_ADC3)
- net GPIO13: now reaches J2.20 (Pin_20)
- net GPIO13: now also U6.17 (GPIO13)
- net GPIO28: now reaches J2.3 (Pin_3)
- net GPIO28: now also U6.42 (GPIO28_ADC2)
- net GPIO26: now reaches J2.5 (Pin_5)
- net GPIO26: now also U6.40 (GPIO26_ADC0)
- net GPIO23: now reaches J2.8 (Pin_8)
- net GPIO23: now also U6.35 (GPIO23)
- net GPIO22: now reaches J2.9 (Pin_9)
- net GPIO22: now also U6.34 (GPIO22)
- net GPIO5: now reaches J1.10 (Pin_10)
- net GPIO5: now also U6.8 (GPIO5)
- net GPIO6: now reaches J1.12 (Pin_12)
- net GPIO6: now also U6.9 (GPIO6)
- net GPIO7: now reaches J1.13 (Pin_13)
- net GPIO7: now also U6.10 (GPIO7)
- net GPIO8: now reaches J1.14 (Pin_14)
- net GPIO8: now also U6.12 (GPIO8)
- net GPIO9: now reaches J1.15 (Pin_15)
- net GPIO9: now also U6.13 (GPIO9)
- net GPIO10: now reaches J1.17 (Pin_17)
- net GPIO10: now also U6.14 (GPIO10)
- net GPIO0: now reaches J1.4 (Pin_4)
- net GPIO0: now also U6.2 (GPIO0)
- net GPIO1: now reaches J1.5 (Pin_5)
- net GPIO1: now also U6.3 (GPIO1)
- net GPIO2: now reaches J1.7 (Pin_7)
- net GPIO2: now also U6.4 (GPIO2)
- net GPIO3: now reaches J1.8 (Pin_8)
- net GPIO3: now also U6.5 (GPIO3)
- net GPIO4: now reaches J1.9 (Pin_9)
- net GPIO4: now also U6.7 (GPIO4)
- net GPIO27: now reaches U6.41 (GPIO27_ADC1)
Other:
- moved on the sheet: SW3, SW4

Commit message: readme
Parts:
- D1: footprint LED_SMD:LED_0402_1005Metric -> LED_SMD:LED_0603_1608Metric
Changed lines of the file:
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@@
 			)
 		)
-		(property "Footprint" "LED_SMD:LED_0402_1005Metric"
+		(property "Footprint" "LED_SMD:LED_0603_1608Metric"
 			(at 288.29 114.3 0)
 			(effects
