File: kicad/_autosave-devboardrp2040.kicad_sch (KiCad schematic)
At the start: 41 parts, among them J1 Conn_01x12_Pin, J2 Conn_01x12_Pin, SW1 SW_Push, SW2 SW_Push, U1 AP63203WU-7, U2 GT-USB-7010ASV, U4 W25Q64JVSSIQ_C179171, U5 ABM8-272-T3_C20625731, U6 RP2350A-QFN60

Commit message: hiii
Connections:
- net +1V1: no longer U6.23 (DVDD), U6.39 (DVDD), U6.50 (VREG_FB), U6.6 (DVDD)
- net +3V3: no longer U6.1 (IOVDD), U6.44 (ADC_AVDD), U6.49 (VREG_VIN)
- net GND: no longer U6.47 (VREG_PGND)
- net GPIO11: no longer U6.15 (GPIO11)
- net GPIO12: no longer U6.16 (GPIO12)
- net GPIO20: no longer U6.32 (GPIO20)
- net GPIO24: no longer U6.36 (GPIO24)
- net IO0: no longer U6.57 (QSPI_SD0)
- net IO1: no longer U6.59 (QSPI_SD1)
- net IO2: no longer U6.58 (QSPI_SD2)
- net IO3: no longer U6.55 (QSPI_SD3)
- net RUN: no longer U6.26 (RUN)
- net VREG_LX: no longer U6.48 (VREG_LX)
- net XIN: no longer U6.21 (XIN)
- net XOUT: no longer U6.22 (XOUT)
- net at J1.10 (Pin_10): now also U6.55 (QSPI_SD3); no longer U6.12 (GPIO8)
- net at J1.11 (Pin_11): no longer U6.13 (GPIO9)
- net at J1.2 (Pin_2): now also U6.48 (VREG_LX); no longer U6.2 (GPIO0)
- net at J1.3 (Pin_3): now also U6.47 (VREG_PGND); no longer U6.3 (GPIO1)
- net at J1.4 (Pin_4): no longer U6.4 (GPIO2)
- net at J1.5 (Pin_5): no longer U6.5 (GPIO3)
- net at J1.6 (Pin_6): no longer U6.7 (GPIO4)
- net at J1.7 (Pin_7): now also U6.57 (QSPI_SD0); no longer U6.8 (GPIO5)
- net at J1.8 (Pin_8): now also U6.59 (QSPI_SD1); no longer U6.9 (GPIO6)
- net at J1.9 (Pin_9): now also U6.58 (QSPI_SD2); no longer U6.10 (GPIO7)
- net at R7.1: no longer U6.52 (USB_DP)
- net at J2.2 (Pin_2): no longer U6.43 (GPIO29_ADC3)
- net at J2.3 (Pin_3): no longer U6.42 (GPIO28_ADC2)
- net at J2.4 (Pin_4): no longer U6.41 (GPIO27_ADC1)
- net at J2.5 (Pin_5): no longer U6.40 (GPIO26_ADC0)
- net at C7.2, R2.2: no longer U6.46 (VREG_AVDD)
- net at R6.2: no longer U6.51 (USB_DM)
- net at U6.56 (QSPI_SCLK): no longer U4.6 (CLK)
Other:
- moved on the sheet: U6
Changed lines of the file:
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@@
 	)
 	(junction
+		(at 270.51 50.8)
+		(diameter 0)
+		(color 0 0 0 0)
+	)
+	(junction
+		(at 270.51 71.12)
+		(diameter 0)
+		(color 0 0 0 0)
+	)
+	(junction
 		(at 167.64 100.33)
 		(diameter 0)
@@
 	)
 	(junction
+		(at 270.51 53.34)
+		(diameter 0)
+		(color 0 0 0 0)
+	)
+	(junction
 		(at 49.53 157.48)
 		(diameter 0)
@@
 	)
 	(junction
+		(at 270.51 63.5)
+		(diameter 0)
+		(color 0 0 0 0)
+	)
+	(junction
 		(at 205.74 -25.4)
 		(diameter 0)
@@
 	)
 	(junction
+		(at 270.51 66.04)
+		(diameter 0)
+		(color 0 0 0 0)
+	)
+	(junction
 		(at 342.9 -27.94)
 		(diameter 0)
@@
 	)
 	(junction
+		(at 270.51 68.58)
+		(diameter 0)
+		(color 0 0 0 0)
+	)
+	(junction
 		(at 205.74 -44.45)
 		(diameter 0)
@@
 	(wire
 		(pts
-			(xy 269.24 50.8) (xy 294.64 50.8)
+			(xy 269.24 50.8) (xy 270.51 50.8)
 		)
 		(stroke
@@
 	(wire
 		(pts
-			(xy 269.24 68.58) (xy 294.64 68.58)
+			(xy 269.24 68.58) (xy 270.51 68.58)
 		)
 		(stroke
@@
 	(wire
 		(pts
+			(xy 270.51 66.04) (xy 294.64 66.04)
+		)
+		(stroke
+			(width 0)
+			(type default)
+		)
+	)
+	(wire
+		(pts
 			(xy 142.24 50.8) (xy 142.24 55.88)
 		)
@@
 	(wire
 		(pts
+			(xy 270.51 50.8) (xy 294.64 50.8)
+		)
+		(stroke
+			(width 0)
+			(type default)
+		)
+	)
+	(wire
+		(pts
+			(xy 270.51 63.5) (xy 294.64 63.5)
+		)
+		(stroke
+			(width 0)
+			(type default)
+		)
+	)
+	(wire
+		(pts
 			(xy 218.44 -44.45) (xy 218.44 -36.83)
 		)
@@
 	(wire
 		(pts
-			(xy 269.24 66.04) (xy 294.64 66.04)
+			(xy 269.24 66.04) (xy 270.51 66.04)
 		)
 		(stroke
@@
 	(wire
 		(pts
-			(xy 269.24 71.12) (xy 294.64 71.12)
+			(xy 269.24 71.12) (xy 270.51 71.12)
 		)
 		(stroke
@@
 	(wire
 		(pts
-			(xy 269.24 63.5) (xy 294.64 63.5)
+			(xy 270.51 71.12) (xy 294.64 71.12)
+		)
+		(stroke
+			(width 0)
+			(type default)
+		)
+	)
+	(wire
+		(pts
+			(xy 269.24 63.5) (xy 270.51 63.5)
 		)
 		(stroke
@@
 	(wire
 		(pts
+			(xy 270.51 68.58) (xy 294.64 68.58)
+		)
+		(stroke
+			(width 0)
+			(type default)
+		)
+	)
+	(wire
+		(pts
 			(xy 297.18 -27.94) (xy 308.61 -27.94)
 		)
@@
 	(wire
 		(pts
-			(xy 269.24 53.34) (xy 294.64 53.34)
+			(xy 269.24 53.34) (xy 270.51 53.34)
 		)
 		(stroke
@@
 	(wire
 		(pts
+			(xy 270.51 53.34) (xy 294.64 53.34)
+		)
+		(stroke
+			(width 0)
+			(type default)
+		)
+	)
+	(wire
+		(pts
 			(xy 308.61 -20.32) (xy 320.04 -20.32)
 		)
@@
 		(lib_id "RPI:RP2350A-QFN60")
 		(at 238.76 78.74 0)
+		(mirror y)
 		(unit 1)
 		(exclude_from_sim no)
@@
 		(on_board yes)
 		(dnp no)
-		(fields_autoplaced yes)
 		(property "Reference" "U6"
-			(at 240.9033 133.35 0)
+			(at 236.6167 133.35 0)
 			(effects
 				(font
@@
 		)
 		(property "Value" "RP2350A-QFN60"
-			(at 240.9033 135.89 0)
+			(at 236.6167 135.89 0)
 			(effects
 				(font
@@
 		)
 		(property "Footprint" "Package_DFN_QFN:QFN-60-1EP_7x7mm_P0.4mm_EP3.4x3.4mm"
-			(at 227.33 60.96 0)
+			(at 250.19 60.96 0)
 			(effects
 				(font
@@
 		)
 		(property "Datasheet" ""
-			(at 227.33 60.96 0)
+			(at 250.19 60.96 0)
 			(effects
 				(font
@@
 		)
 		(property "Description" ""
-			(at 232.41 64.77 0)
+			(at 245.11 64.77 0)
 			(effects
 				(font
