File: kicad/_autosave-devboardrp2040.kicad_pcb (KiCad board)
At the start: 4 copper layers, 59.2 x 26.4 mm, 43 parts, among them J1 Conn_01x23_Pin, J2 Conn_01x23_Pin, SW1 SW_Push, SW3 SW_Push, SW4 SW_Push, U1 AP63203WU-7, U2 GT-USB-7010ASV, U4 W25Q64JVSSIQ_C179171, U5 ABM8-272-T3_C20625731, U6 RP2350A-QFN60

Commit message: silkscreen!!!
Parts:
- added G***: LOGO, LOGO, F.Cu at (150.8, 73.3)
Routing:
- net RUN: track 44.0 -> 45.2 mm
Other:
- board text added: "@spc"
- board text added: "^-^"
- board text added: "clicky"
- board text added: "gpio11 + boot"
- board text added: "gpio17"
- board text added: "gpio18"
- board text added: "gpio25"
- board text added: "mx cherry here x3"
- board text added: "rp2350a!!"
- board text added: "usb 7.4"
- board text added: "use your coolest caps"
