File: kicad/v1.0-pcb/devbackup.kicad_pcb (KiCad board)
At the start: 2 copper layers, 31.5 x 25.5 mm, 41 parts, among them J1 Conn_01x12_Pin, J2 Conn_01x12_Pin, SW1 SW_Push, SW2 SW_Push, U1 AP63203WU-7, U2 GT-USB-7010ASV, U4 W25Q64JVSSIQ_C179171, U5 ABM8-272-T3_C20625731, U6 RP2350A-QFN60

Commit message: hiii
Parts:
- moved U2 0.98 mm to (77.8, 42.4)
Routing:
- net D-: track 7.73 -> 9.69 mm
- net USB_VBUS: track 37.3 -> 39.2 mm
- net Net-(U2-CC1): track 4.82 -> 5.80 mm
- net D+: track 8.35 -> 9.26 mm
- net GND: vias 28 -> 30
Other:
- board size 31.5 x 25.5 mm -> 33.6 x 25.4 mm
Changed lines of the file:
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@@
 	(footprint "easyeda2kicad:USB-C-SMD_G-SWITCH_GT-USB-7010ASV"
 		(layer "F.Cu")
-		(at 76.8 42.43 90)
+		(at 77.775 42.425 90)
 		(property "Reference" "U2"
 			(at 3.755 27.155 90)
@@
 	)
 	(gr_arc
-		(start 48.75 31.75)
-		(mid 49.335786 30.335786)
-		(end 50.75 29.75)
+		(start 49.725 55.125)
+		(mid 48.310786 54.539214)
+		(end 47.725 53.125)
 		(stroke
 			(width 0.05)
@@
 		(layer "Edge.Cuts")
 	)
-	(gr_line
-		(start 80.25 31.75)
-		(end 80.25 53.2)
+	(gr_arc
+		(start 47.725 31.725)
+		(mid 48.310786 30.310786)
+		(end 49.725 29.725)
 		(stroke
 			(width 0.05)
@@
 		(layer "Edge.Cuts")
 	)
-	(gr_arc
-		(start 78.25 29.75)
-		(mid 79.664214 30.335786)
-		(end 80.25 31.75)
+	(gr_line
+		(start 81.325 31.725)
+		(end 81.325 53.125)
 		(stroke
 			(width 0.05)
@@
 	)
 	(gr_arc
-		(start 80.25 53.2)
-		(mid 79.664214 54.614214)
-		(end 78.25 55.2)
+		(start 81.325 53.125)
+		(mid 80.739214 54.539214)
+		(end 79.325 55.125)
 		(stroke
 			(width 0.05)
@@
 	)
 	(gr_line
-		(start 78.25 55.2)
-		(end 50.75 55.2)
+		(start 47.725 53.125)
+		(end 47.725 31.725)
 		(stroke
 			(width 0.05)
@@
 	)
 	(gr_line
-		(start 48.75 53.2)
-		(end 48.75 31.75)
+		(start 49.725 29.725)
+		(end 79.325 29.725)
 		(stroke
 			(width 0.05)
@@
 		(layer "Edge.Cuts")
 	)
-	(gr_arc
-		(start 50.75 55.2)
-		(mid 49.335786 54.614214)
-		(end 48.75 53.2)
+	(gr_line
+		(start 79.325 55.125)
+		(end 49.725 55.125)
 		(stroke
 			(width 0.05)
@@
 		(layer "Edge.Cuts")
 	)
-	(gr_line
-		(start 50.75 29.75)
-		(end 78.25 29.75)
+	(gr_arc
+		(start 79.325 29.725)
+		(mid 80.739214 30.310786)
+		(end 81.325 31.725)
 		(stroke
 			(width 0.05)
@@
 	)
 	(segment
-		(start 76.47 40.66)
-		(end 76.05 41.08)
+		(start 77.445 40.655)
+		(end 77.025 41.075)
 		(width 0.2)
 		(layer "F.Cu")
@@
 	)
 	(segment
-		(start 74.599 44.631)
-		(end 74.4 44.83)
-		(width 0.2)
-		(layer "F.Cu")
-		(net 1)
-	)
-	(segment
-		(start 76.05 41.08)
-		(end 76.05 43.902)
+		(start 77.025 41.075)
+		(end 77.025 43.897)
 		(width 0.2)
 		(layer "F.Cu")
@@
 	)
 	(segment
-		(start 76.05 43.902)
-		(end 75.321 44.631)
+		(start 77.025 43.897)
+		(end 76.296 44.626)
 		(width 0.2)
 		(layer "F.Cu")
@@
 	)
 	(segment
-		(start 75 40.03)
-		(end 76.05 41.08)
+		(start 75.975 40.025)
+		(end 77.025 41.075)
 		(width 0.2)
 		(layer "F.Cu")
@@
 	)
 	(segment
-		(start 76.47 39.78)
-		(end 76.47 40.66)
+		(start 77.445 39.775)
+		(end 77.445 40.655)
 		(width 0.2)
 		(layer "F.Cu")
@@
 	)
 	(segment
+		(start 74.405 44.825)
+		(end 75.375 44.825)
+		(width 0.2)
+		(layer "F.Cu")
+		(net 1)
+	)
+	(segment
 		(start 72.46 46.27)
 		(end 71.35 46.27)
@@
 	)
 	(segment
-		(start 75.321 44.631)
-		(end 74.599 44.631)
+		(start 76.296 44.626)
+		(end 75.574 44.626)
+		(width 0.2)
+		(layer "F.Cu")
+		(net 1)
+	)
+	(segment
+		(start 74.4 44.83)
+		(end 74.405 44.825)
 		(width 0.2)
 		(layer "F.Cu")
@@
 	)
 	(via
-		(at 76.47 39.78)
+		(at 77.445 39.775)
 		(size 0.4)
 		(drill 0.2)
@@
 	)
 	(segment
-		(start 76.82 36.809)
-		(end 76.47 37.159)
+		(start 76.84 36.815)
+		(end 78.325 38.3)
+		(width 0.2)
+		(layer "B.Cu")
+		(net 1)
+	)
+	(segment
+		(start 77.975 39.775)
+		(end 77.445 39.775)
+		(width 0.2)
+		(layer "B.Cu")
+		(net 1)
+	)
+	(segment
+		(start 78.325 38.3)
+		(end 78.325 39.425)
 		(width 0.2)
 		(layer "B.Cu")
@@
 	)
 	(segment
+		(start 78.325 39.425)
+		(end 77.975 39.775)
+		(width 0.2)
+		(layer "B.Cu")
+		(net 1)
+	)
+	(segment
 		(start 76.84 36.809)
 		(end 76.82 36.809)
@@
 	)
 	(segment
-		(start 76.47 37.159)
-		(end 76.47 39.78)
+		(start 76.84 36.809)
+		(end 76.84 36.815)
 		(width 0.2)
 		(layer "B.Cu")
@@
 	)
 	(segment
+		(start 74.3 43.68)
+		(end 74.4 43.68)
+		(width 0.2)
+		(layer "F.Cu")
+		(net 10)
+	)
+	(segment
 		(start 73.42 43.68)
+		(end 74.3 43.68)
+		(width 0.2)
+		(layer "F.Cu")
+		(net 10)
+	)
+	(segment
+		(start 75.375 43.675)
+		(end 74.405 43.675)
+		(width 0.2)
+		(layer "F.Cu")
+		(net 10)
+	)
+	(segment
+		(start 74.405 43.675)
 		(end 74.4 43.68)
 		(width 0.2)
@@
 	)
 	(segment
+		(start 74.405 42.175)
+		(end 74.4 42.18)
+		(width 0.2)
+		(layer "F.Cu")
+		(net 15)
+	)
+	(segment
+		(start 74.4 43.18)
+		(end 74.405 43.175)
+		(width 0.2)
+		(layer "F.Cu")
+		(net 15)
+	)
+	(segment
 		(start 71.53 43.18)
 		(end 70.13 44.58)
@@
 	)
 	(segment
+		(start 74.405 43.175)
+		(end 75.375 43.175)
+		(width 0.2)
+		(layer "F.Cu")
+		(net 15)
+	)
+	(segment
 		(start 73.43 42.18)
 		(end 73.43 43.082)
@@
 	)
 	(segment
+		(start 75.375 42.175)
+		(end 74.405 42.175)
+		(width 0.2)
+		(layer "F.Cu")
+		(net 15)
+	)
+	(segment
 		(start 73.528 43.18)
 		(end 74.4 43.18)
@@
 	)
 	(segment
-		(start 73.3629 41.68)
-		(end 73.029 42.0139)
+		(start 74.4 41.68)
+		(end 74.405 41.675)
 		(width 0.2)
 		(layer "F.Cu")
@@
 	)
 	(segment
-		(start 74.4 42.68)
-		(end 74.449 42.729)
+		(start 73.3629 41.68)
+		(end 73.029 42.0139)
 		(width 0.2)
 		(layer "F.Cu")
@@
 	)
 	(segment
-		(start 75.272 41.68)
-		(end 74.4 41.68)
+		(start 76.247 41.675)
+		(end 75.375 41.675)
+		(width 0.2)
+		(layer "F.Cu")
+		(net 16)
+	)
+	(segment
+		(start 74.405 41.675)
+		(end 75.375 41.675)
 		(width 0.2)
 		(layer "F.Cu")
@@
 	)
 	(segment
-		(start 75.321 42.729)
-		(end 75.321 41.729)
+		(start 76.296 42.724)
+		(end 76.296 41.724)
 		(width 0.2)
 		(layer "F.Cu")
@@
 	)
 	(segment
-		(start 74.449 42.729)
-		(end 75.321 42.729)
+		(start 75.424 42.724)
+		(end 76.296 42.724)
 		(width 0.2)
 		(layer "F.Cu")
@@
 	)
 	(segment
-		(start 75.321 41.729)
-		(end 75.272 41.68)
+		(start 76.296 41.724)
+		(end 76.247 41.675)
 		(width 0.2)
 		(layer "F.Cu")
@@
 	)
 	(via
+		(at 54.91 45.16)
+		(size 0.6)
+		(drill 0.3)
+		(layers "F.Cu" "B.Cu")
+		(free yes)
+		(net 44)
+	)
+	(via
 		(at 51.78 32.29)
 		(size 0.6)
@@
 	)
 	(via
+		(at 49.84 41.83)
+		(size 0.6)
+		(drill 0.3)
+		(layers "F.Cu" "B.Cu")
+		(free yes)
+		(net 44)
+	)
+	(via
 		(at 53.99 46.51)
 		(size 0.6)
@@
 	)
 	(via
-		(at 75.54 43.42)
+		(at 76.515 43.415)
 		(size 0.4)
 		(drill 0.2)
